File: 05-Schematic/Dirks_IndividualSubsystem.kicad_sch (KiCad schematic)
At the start: 86 parts, among them J1 Barrel_Jack, J2 8 Pin In, J3 8Pin out, M1 Motor_DC, M2 Motor_DC, M3 Motor_DC, M4 Motor_Servo, M5 Motor_Servo

Commit message: deploy: d9f193009c9cfe113089e705a54987470ddf529e
Parts:
- removed C13: 22uF, symbol Device:C_Small
- removed C14: .1uF, symbol Dirks_EGR314:CPWR_Small
- added C29: 22uF, symbol Device:C_Small
- added C30: .1uF, symbol Dirks_EGR314:CPWR_Small
- C4: value n/a -> .47uF
Connections:
- net +3.3V: now also U1.2 (3V3), C29.1, C30.2
- net GND: now also C1.2, C3.2, C29.2, C30.1

Commit message: deploy: d75c61953b70b9b3690e90ed7fc4e2a405ae5d79
Parts:
- added D4, D5, D6: D, symbol Device:D
- added F2: Fuse 3.5 A, symbol Device:Fuse
- added R9: 10K, symbol Device:R_US
- added SW1: SW_DPST, symbol Switch:SW_DPST
- added TP1, TP2, TP32, TP33, TP34, TP35, TP6: TestPoint_Small, symbol Connector:TestPoint_Small
Connections:
- net +3.3V: now also D6.1 (K), SW1.2; no longer C7.1, C9.1, L1.2
- net +5V: now also D4.1 (K); no longer C15.1, C16.1, L2.2, R4.2, VR2.12 (Out)
- net GND: now also R9.1
- net MISO: now also TP6.1
- net MOSI: now also TP2.1
- net VDC: no longer J2.7, J3.7
- net chip select: no longer U1.18 (IO10), U3.9 (CSN), U4.9 (CSN)
- net at J3.1: now also TP33.1
- net at J3.2: now also TP34.1
- net at J3.3: now also TP35.1
- net at TP7.1: now also J2.6; no longer U1.15 (IO3)
- net at U3.8 (SI), U4.3 (SO): now also TP1.1
- net +12V: now reaches F1.1, J1.1
- net +12V: now also D5.2 (A)
- net at U1.33 (IO40): now also R9.2, SW1.1; no longer TP23.1
- net at TP8.1: now also J2.5; no longer U1.16 (IO46)
- net at J2.1: now also TP32.1
- net at J2.2: now also TP23.1
- new net: C7.1, C9.1, D6.2 (A), L1.2
- new net: D5.1 (K), F2.2
- new net: C15.1, C16.1, D4.2 (A), L2.2, R4.2, VR2.12 (Out)
- new net chip select1: U1.18 (IO10)
- new net chip select2: U1.16 (IO46), U4.9 (CSN)
- new net chip select3: U1.15 (IO3), U3.9 (CSN)
- new net shareLine: F2.1, J2.7, J3.7
- no-connect marks 29 -> 24
Other:
- moved on the sheet: C18, C21, D3, F1

Commit message: deploy: c582b7a0318d92a64421fd9f42b441bc38769731
Parts:
- removed C20: 100uF, symbol Device:C_Small
- removed C22: 100nF, symbol Device:C_Small
- removed D3, D4, D5, D6: D, symbol Device:D
- removed M4: Motor_Servo, symbol Motor:Motor_Servo
- removed R9: 10K, symbol Device:R_US
- removed TP18, TP19, TP20, TP28, TP8: TestPoint_Small, symbol Connector:TestPoint_Small
- added C17, C19, C29, C31: 100uF, Capacitor_SMD:C_1210_3225Metric, symbol Device:C_Small
- added C30, C32: 100nF, Capacitor_SMD:C_0201_0603Metric, symbol Device:C_Small
- added D2, D3, D4, D6: D, Package_TO_SOT_SMD:TO-252-3_TabPin2, symbol Device:D_Schottky_AKA
- added M1: Motor_Servo, Dirks_EGR314Library:3PinScrewTerminal, symbol Motor:Motor_Servo
- added R6, R7: 10K, Resistor_SMD:R_2512_6332Metric, symbol Device:R_US
- added SW2: SW_DPST, Dirks_EGR314Library:standardPushButton, symbol Switch:SW_DPST
- added TP15, TP16, TP17, TP35: TestPoint_Small, Connector_PinHeader_2.54mm:PinHeader_1x01_P2.54mm_Vertical, symbol Connector:TestPoint_Small
- C1: renamed from C2; footprint (none) -> Capacitor_SMD:C_01005_0402Metric
- C10: renamed from C12; footprint (none) -> Capacitor_SMD:C_0201_0603Metric
- C11: renamed from C8; footprint (none) -> Capacitor_SMD:C_0201_0603Metric
- C12: renamed from C9; footprint (none) -> Capacitor_SMD:C_01005_0402Metric
- C13: renamed from C15; footprint (none) -> Capacitor_SMD:C_1210_3225Metric
- C14: renamed from C16; footprint (none) -> Capacitor_SMD:C_01005_0402Metric
- C15: renamed from C29; value 22uF -> 22 uF; footprint (none) -> Capacitor_SMD:C_01005_0402Metric
- C16: renamed from C30; value .1uF -> 100nF; footprint (none) -> Capacitor_SMD:C_0201_0603Metric
- C18: value 100uF -> 100nF; footprint (none) -> Capacitor_SMD:C_0201_0603Metric
- C2: renamed from C1; footprint (none) -> Capacitor_SMD:C_0603_1608Metric
- C20: renamed from C17; footprint (none) -> Capacitor_SMD:C_1210_3225Metric
- C21, C4, C5: footprint (none) -> Capacitor_SMD:C_0201_0603Metric
- C22: renamed from C19; footprint (none) -> Capacitor_SMD:C_0201_0603Metric
- C23, C24, C25, C26, C27, C28, C6: footprint (none) -> Capacitor_SMD:C_0805_2012Metric
- C3: footprint (none) -> Capacitor_SMD:C_0603_1608Metric
- C7: renamed from C10; footprint (none) -> Capacitor_SMD:C_01005_0402Metric
- C8: renamed from C11; footprint (none) -> Capacitor_SMD:C_0201_0603Metric
- C9: renamed from C7; footprint (none) -> Capacitor_SMD:C_01005_0402Metric
- D1: footprint (none) -> Package_TO_SOT_SMD:TO-252-3_TabPin2; symbol Device:D -> Device:D_Schottky_AKA
- D5: renamed from D2; footprint (none) -> LED_SMD:LED_0805_2012Metric
- F1, F2: footprint (none) -> Dirks_EGR314Library:FUSE_4628
- J1: footprint (none) -> Dirks_EGR314Library:PJ-102AH_CUD
- J2: renamed from J4; footprint (none) -> Dirks_EGR314Library:CONN_USB3131-30-0230-A_GCT
- J3: renamed from J2; footprint CONN_7024608xx_MOL -> Dirks_EGR314Library:CONN_332LF_AMP
- J4: renamed from J3; footprint CONN_7024608xx_MOL -> Dirks_EGR314Library:CONN_332LF_AMP
- L1: renamed from L2; footprint (none) -> Dirks_EGR314Library:33uFInductor
- L2: renamed from L1; footprint (none) -> Dirks_EGR314Library:47uFInductor
- M2: renamed from M5; footprint (none) -> Dirks_EGR314Library:3PinScrewTerminal
- M3: renamed from M1; footprint (none) -> Dirks_EGR314Library:2PinScrewTerminal
- M4: renamed from M2; footprint (none) -> Dirks_EGR314Library:2PinScrewTerminal
- M5: renamed from M3; footprint (none) -> Dirks_EGR314Library:2PinScrewTerminal
- R1, R2, R4, R5: footprint (none) -> Resistor_SMD:R_2512_6332Metric
- R10: renamed from R7; footprint (none) -> Resistor_SMD:R_2512_6332Metric
- R11: renamed from R6; footprint (none) -> Resistor_SMD:R_2512_6332Metric
- R3: footprint (none) -> Resistor_SMD:R_1206_3216Metric
- R9: renamed from R8; footprint (none) -> Resistor_SMD:R_2512_6332Metric
- S1: footprint (none) -> Dirks_EGR314Library:fancyBTN_DPDT_TL2233_EWI
- SW1: footprint (none) -> Dirks_EGR314Library:standardPushButton
- TP1, TP29: footprint (none) -> Connector_PinHeader_2.54mm:PinHeader_1x01_P2.54mm_Vertical
- TP10: renamed from TP15; footprint (none) -> Connector_PinHeader_2.54mm:PinHeader_1x01_P2.54mm_Vertical
- TP11: renamed from TP16; footprint (none) -> Connector_PinHeader_2.54mm:PinHeader_1x01_P2.54mm_Vertical
- TP12: renamed from TP17; footprint (none) -> Connector_PinHeader_2.54mm:PinHeader_1x01_P2.54mm_Vertical
- TP13: renamed from TP6; footprint (none) -> Connector_PinHeader_2.54mm:PinHeader_1x01_P2.54mm_Vertical
- TP14: renamed from TP2; footprint (none) -> Connector_PinHeader_2.54mm:PinHeader_1x01_P2.54mm_Vertical
- TP18: renamed from TP21; footprint (none) -> Connector_PinHeader_2.54mm:PinHeader_1x01_P2.54mm_Vertical
- TP19: renamed from TP22; footprint (none) -> Connector_PinHeader_2.54mm:PinHeader_1x01_P2.54mm_Vertical
- TP2: renamed from TP3; footprint (none) -> Connector_PinHeader_2.54mm:PinHeader_1x01_P2.54mm_Vertical
- TP20: renamed from TP24; footprint (none) -> Connector_PinHeader_2.54mm:PinHeader_1x01_P2.54mm_Vertical
- TP21: renamed from TP25; footprint (none) -> Connector_PinHeader_2.54mm:PinHeader_1x01_P2.54mm_Vertical
- TP22: renamed from TP26; footprint (none) -> Connector_PinHeader_2.54mm:PinHeader_1x01_P2.54mm_Vertical
- TP23: renamed from TP27; footprint (none) -> Connector_PinHeader_2.54mm:PinHeader_1x01_P2.54mm_Vertical
- TP25: renamed from TP5; footprint (none) -> Connector_PinHeader_2.54mm:PinHeader_1x01_P2.54mm_Vertical
- TP26: renamed from TP31; footprint (none) -> Connector_PinHeader_2.54mm:PinHeader_1x01_P2.54mm_Vertical
- TP27: renamed from TP32; footprint (none) -> Connector_PinHeader_2.54mm:PinHeader_1x01_P2.54mm_Vertical
- TP28: renamed from TP23; footprint (none) -> Connector_PinHeader_2.54mm:PinHeader_1x01_P2.54mm_Vertical
- TP3: renamed from TP4; footprint (none) -> Connector_PinHeader_2.54mm:PinHeader_1x01_P2.54mm_Vertical
- TP30: renamed from TP7; footprint (none) -> Connector_PinHeader_2.54mm:PinHeader_1x01_P2.54mm_Vertical
- TP31: renamed from TP33; footprint (none) -> Connector_PinHeader_2.54mm:PinHeader_1x01_P2.54mm_Vertical
- TP32: renamed from TP34; footprint (none) -> Connector_PinHeader_2.54mm:PinHeader_1x01_P2.54mm_Vertical
- TP33: renamed from TP35; footprint (none) -> Connector_PinHeader_2.54mm:PinHeader_1x01_P2.54mm_Vertical
- TP34: renamed from TP30; footprint (none) -> Connector_PinHeader_2.54mm:PinHeader_1x01_P2.54mm_Vertical
- TP4: renamed from TP9; footprint (none) -> Connector_PinHeader_2.54mm:PinHeader_1x01_P2.54mm_Vertical
- TP5: renamed from TP10; footprint (none) -> Connector_PinHeader_2.54mm:PinHeader_1x01_P2.54mm_Vertical
- TP6: renamed from TP11; footprint (none) -> Connector_PinHeader_2.54mm:PinHeader_1x01_P2.54mm_Vertical
- TP7: renamed from TP12; footprint (none) -> Connector_PinHeader_2.54mm:PinHeader_1x01_P2.54mm_Vertical
- TP8: renamed from TP13; footprint (none) -> Connector_PinHeader_2.54mm:PinHeader_1x01_P2.54mm_Vertical
- TP9: renamed from TP14; footprint (none) -> Connector_PinHeader_2.54mm:PinHeader_1x01_P2.54mm_Vertical
- U1: renamed from U2; footprint Dirks_EGR314Library:IFX9201SGAUMA1_footprint -> Dirks_EGR314Library:MotorDriver_IFX9201SGAUMA1
- U2: renamed from U3; footprint Dirks_EGR314Library:IFX9201SGAUMA1_footprint -> Dirks_EGR314Library:MotorDriver_IFX9201SGAUMA1
- U3: renamed from U4; footprint Dirks_EGR314Library:IFX9201SGAUMA1_footprint -> Dirks_EGR314Library:MotorDriver_IFX9201SGAUMA1
- U4: renamed from U1; footprint (none) -> Dirks_EGR314Library:n8ESP32-S3-WROOM-1_EXP
- VR1: renamed from VR2; footprint Dirks_EGR314Library:LM5005MHXNOPB_Buck2_5A -> Dirks_EGR314Library:Buck2_5LM5005MHXNOPB
- VR2: renamed from VR1; footprint Dirks_EGR314Library:AP63203WU-7_Buck2A -> Dirks_EGR314Library:Buck2A_AP63203WU-7
Connections:
- net VDC is gone; now on net 12vL: F1.2
- net chip select is gone; now on net chip select1: U1.9 (CSN)
- net +12V: now also D4.3 (A)
- net +3.3V: now also TP29.1, C31.1, C32.1, D2.2 (K), R6.1, R7.1; no longer C18.1, C20.1, C21.1, C22.1, SW1.2
- net +5V: now also C18.1, C20.1, C21.1, C22.1, U1.2 (VSO), U1.4 (VS), U2.2 (VSO), U2.4 (VS), U3.2 (VSO), U3.4 (VS), C17.1, C19.1, C29.1, C30.1, D3.2 (K), M1.2 (+), TP17.1
- net GND: now also C18.2, C20.2, C21.2, C22.2, S1.3, S1.6, SW1.2, SW1.4, U4.41 (GND), U4.42 (GND), U4.43 (GND), U4.44 (GND), U4.45 (GND), U4.46 (GND), U4.47 (GND), U4.48 (GND), U4.49 (GND), C17.2, C19.2, C29.2, C30.2, C31.2, C32.2, M1.3 (-), SW2.2, SW2.4, TP15.1, TP16.1, TP35.1
- net MISO: now also U2.3 (SO); no longer U1.8 (SI)
- net MOSI: now also U1.8 (SI); no longer U2.3 (SO)
- net UartIn: now also J3.5, D6.1 (A); no longer J3.4
- net UartOut: now also D6.2 (K)
- net chip select1: now also U4.22 (IO14); no longer U4.18 (IO10)
- net chip select2: now also U4.23 (IO21); no longer U4.16 (IO46)
- net chip select3: now also U4.24 (IO47); no longer U4.15 (IO3)
- net pwm1: now also M1.1 (PWM)
- net at C12.1, C9.1, L2.2: now also D2.1 (A), D2.3 (A)
- net at SW1.1: now also SW1.3, U4.3 (EN), R6.2; no longer U4.33 (IO40)
- net at F2.2: now also D4.2 (K)
- net at C13.1, C14.1, L1.2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: now also D3.3 (A)
- net 12vL: now reaches C2.1, C3.1, VR1.3 (VIN)
- net 12vL: now also C6.1, VR2.2 (EN), VR2.3 (VIN)
- net at VR1.15 (IS): now also D1.3 (A); no longer D1.2 (A)
- net at C10.1, C8.2, L1.1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: now also D1.2 (K); no longer D1.1 (K)
- net at R11.1: now also S1.4; no longer S1.6
- net at U4.27 (IO0): now also R7.2, SW2.1, SW2.3; no longer TP29.1
- no-connect marks 24 -> 31
Other:
- note added: "Necessary for Kicad to be happy regarding lines where 5v and 3.3v are either entering the system or exiting."
- moved on the sheet: C10, C15, C16, C20, C22, C23, C24, C25, C26, C27, C28, C6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

Commit message: deploy: 0fce7d7e37bb53a5a80ff59e97df34172e537118
Parts:
- removed TP28, TP32: TestPoint_Small, Connector_PinHeader_2.54mm:PinHeader_1x01_P2.54mm_Vertical, symbol Connector:TestPoint_Small
Connections:
- net UartIn: now also J3.2; no longer J3.5
- net UartOut: now also J4.2; no longer J4.5
- no-connect marks 31 -> 32
Other:
- moved on the sheet: D6
Changed lines of the file:
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@@
 	)
 	(no_connect
-		(at 259.08 26.67)
+		(at 259.08 29.21)
 	)
 	(no_connect
@@
 	)
 	(no_connect
+		(at 259.08 26.67)
+	)
+	(no_connect
 		(at 175.26 53.34)
 	)
@@
 	)
 	(no_connect
-		(at 246.38 49.53)
+		(at 246.38 40.64)
 	)
 	(no_connect
@@
 	)
 	(no_connect
+		(at 259.08 24.13)
+	)
+	(no_connect
 		(at 125.73 40.64)
 	)
@@
 	)
 	(no_connect
-		(at 259.08 24.13)
-	)
-	(no_connect
 		(at 172.72 25.4)
 	)
@@
 	(wire
 		(pts
-			(xy 259.08 50.8) (xy 256.54 50.8)
-		)
-		(stroke
-			(width 0)
-			(type default)
-		)
-	)
-	(wire
-		(pts
 			(xy 67.31 163.83) (xy 54.61 163.83)
 		)
@@
 	(wire
 		(pts
-			(xy 243.84 29.21) (xy 243.84 49.53)
+			(xy 243.84 21.59) (xy 243.84 40.64)
 		)
 		(stroke
@@
 	(wire
 		(pts
-			(xy 74.93 35.56) (xy 76.2 35.56)
+			(xy 246.38 50.8) (xy 246.38 49.53)
 		)
 		(stroke
@@
 	(wire
 		(pts
-			(xy 259.08 21.59) (xy 256.54 21.59)
+			(xy 74.93 35.56) (xy 76.2 35.56)
 		)
 		(stroke
@@
 	(wire
 		(pts
-			(xy 243.84 29.21) (xy 259.08 29.21)
+			(xy 243.84 21.59) (xy 259.08 21.59)
 		)
 		(stroke
@@
 	(wire
 		(pts
-			(xy 246.38 58.42) (xy 259.08 58.42)
+			(xy 246.38 50.8) (xy 259.08 50.8)
 		)
 		(stroke
@@
 	)
 	(label "UartOut"
-		(at 251.46 58.42 0)
+		(at 250.19 50.8 0)
 		(effects
 			(font
@@
 	)
 	(label "UartIn"
-		(at 246.38 29.21 0)
+		(at 246.38 21.59 0)
 		(effects
 			(font
@@
 		(dnp no)
 		(property "Reference" "TP27"
-			(at 254.762 19.558 0)
+			(at 256.54 17.272 0)
 			(effects
 				(font
@@
 		(dnp no)
 		(property "Reference" "TP31"
-			(at 254.762 48.768 0)
+			(at 257.556 47.244 0)
 			(effects
 				(font
@@
 	(symbol
 		(lib_id "Connector:TestPoint_Small")
-		(at 256.54 21.59 180)
-		(unit 1)
-		(exclude_from_sim no)
-		(in_bom yes)
-		(on_board yes)
-		(dnp no)
-		(property "Reference" "TP28"
-			(at 254.762 22.098 0)
-			(effects
-				(font
-					(size 1.27 1.27)
-				)
-				(justify left)
-			)
-		)
-		(property "Value" "TestPoint_Small"
-			(at 255.27 20.3201 0)
-			(effects
-				(font
-					(size 1.27 1.27)
-				)
-				(justify left)
-				(hide yes)
-			)
-		)
-		(property "Footprint" "Connector_PinHeader_2.54mm:PinHeader_1x01_P2.54mm_Vertical"
-			(at 251.46 21.59 0)
-			(effects
-				(font
-					(size 1.27 1.27)
-				)
-				(hide yes)
-			)
-		)
-		(property "Datasheet" "~"
-			(at 251.46 21.59 0)
-			(effects
-				(font
-					(size 1.27 1.27)
-				)
-				(hide yes)
-			)
-		)
-		(property "Description" "test point"
-			(at 256.54 21.59 0)
-			(effects
-				(font
-					(size 1.27 1.27)
-				)
-				(hide yes)
-			)
-		)
-		(pin "1"
-		)
-		(instances
-			(project "Dirks_IndividualSubsystem"
-				(path "/b9dc885c-c6d6-4e3b-ba8a-e6588a4501d6"
-					(reference "TP28")
-					(unit 1)
-				)
-			)
-		)
-	)
-	(symbol
-		(lib_id "Connector:TestPoint_Small")
 		(at 236.22 92.71 180)
 		(unit 1)
@@
 	(symbol
 		(lib_id "Device:D_Schottky_AKA")
-		(at 246.38 54.61 90)
+		(at 246.38 45.72 90)
 		(unit 1)
 		(exclude_from_sim no)
@@
 		(dnp no)
 		(property "Reference" "D6"
-			(at 244.094 55.626 0)
+			(at 244.094 46.736 0)
 			(effects
 				(font
@@
 		)
 		(property "Value" "D"
-			(at 249.174 52.832 0)
+			(at 249.174 43.942 0)
 			(effects
 				(font
@@
 		)
 		(property "Footprint" "Package_TO_SOT_SMD:TO-252-3_TabPin2"
-			(at 246.38 54.61 0)
+			(at 246.38 45.72 0)
 			(effects
 				(font
@@
 		)
 		(property "Datasheet" "~"
-			(at 246.38 54.61 0)
+			(at 246.38 45.72 0)
 			(effects
 				(font
@@
 		)
 		(property "Description" "Schottky diode, anode on pins 1 and 3"
-			(at 246.38 54.61 0)
+			(at 246.38 45.72 0)
 			(effects
 				(font
@@
 		)
 		(property "Sim.Device" "D"
-			(at 246.38 54.61 0)
+			(at 246.38 45.72 0)
 			(effects
 				(font
@@
 		)
 		(property "Sim.Pins" "1=K 2=A"
-			(at 246.38 54.61 0)
+			(at 246.38 45.72 0)
 			(effects
 				(font
@@
 					(unit 1)
 				)
-			)
-		)
-	)
-	(symbol
-		(lib_id "Connector:TestPoint_Small")
-		(at 256.54 50.8 180)
-		(unit 1)
-		(exclude_from_sim no)
-		(in_bom yes)
-		(on_board yes)
-		(dnp no)
-		(property "Reference" "TP32"
-			(at 254.762 51.308 0)
-			(effects
-				(font
-					(size 1.27 1.27)
-				)
-				(justify left)
-			)
-		)
-		(property "Value" "TestPoint_Small"
-			(at 255.27 49.5301 0)
-			(effects
-				(font
-					(size 1.27 1.27)
-				)
-				(justify left)
-				(hide yes)
-			)
-		)
-		(property "Footprint" "Connector_PinHeader_2.54mm:PinHeader_1x01_P2.54mm_Vertical"
-			(at 251.46 50.8 0)
-			(effects
-				(font
-					(size 1.27 1.27)
-				)
-				(hide yes)
-			)
-		)
-		(property "Datasheet" "~"
-			(at 251.46 50.8 0)
-			(effects
-				(font
-					(size 1.27 1.27)
-				)
-				(hide yes)
-			)
-		)
-		(property "Description" "test point"
-			(at 256.54 50.8 0)
-			(effects
-				(font
-					(size 1.27 1.27)
-				)
-				(hide yes)
-			)
-		)
-		(pin "1"
-		)
-		(instances
-			(project "Dirks_IndividualSubsystem"
-				(path "/b9dc885c-c6d6-4e3b-ba8a-e6588a4501d6"
-					(reference "TP32")
-					(unit 1)
-				)
